File: Circuit/Starlings Technology nrf52.sch (EAGLE design)
At the start: 49 parts, among them IC1 MCP1703CB, J4 USB Micro, J7 CORTEX_DEBUG_SMD, Q2 BSS84, U1 TPS61032PWP, U2 MCP73831, U3 BC840M, U5 74AHCT2G125, Y2 FC-12M

Commit message: Revision 12, changes out buttons and resistors.
- PTH tactile switches for taller buttons
- Resistor array and digikey swap
Parts:
- removed R14, R5: 1k, SparkFun-Resistors:1KOHM-0603-1/10W-1%
- removed R4, R6: 330, SparkFun:RESISTOR0603-RES
- removed RN1: 100K, resistor-dil:4R-NEXB38V
- added R1: 100k, SparkFun:RESISTOR0603-RES
- added RN2: (no value), resistor-dil:4R-NEXBS8V
- C3: value 220µF -> 220uF; device SparkFun-Capacitors:10UF-POLAR-EIA6032-25V-10% -> SparkFun-Capacitors:47UF-POLAR-EIA3528-10V-10%
- Q2: DIGIKEY DMG2301L-7DITR-ND -> DMP2215LDICT-ND
- R15: DIGIKEY 311-22.0HRTR-ND -> 311-22.0HRCT-ND
- RPROG: value 2.0k -> 5.0k; DIGIKEY ‎311-2.00KHRCT-ND‎ -> RMCF0603JT2K00CT-ND
- U2: DIGIKEY MCP73831T-2ACI/OTTR-ND -> 497-5809-1-ND
Connections:
- net 3.3V: now also RN2A.1, RN2B.1; no longer R4.1, R6.2
- net GND: now also R1.1, RN2D.1; no longer R14.2, RN1A.1
- net N$1: now also RN2A.2; no longer R4.2
- net N$13: now also RN2D.2; no longer R14.1
- net N$15: now also RN2C.2; no longer R5.1
- net N$8: now also RN2B.2; no longer R6.1
- net VBUS: now also R1.2, RN2C.1; no longer R5.2, RN1A.2
Other:
- note added: "Revision history: 2022-04-28: Revision 12 - PTH tactile switches for taller buttons - Resistor array and digikey swap 2022-04-12: Revision 11 - Switching boost converter and inductor 2022-03-11: Revision 10 - Adding second tactile switch - Adjusting board dimensions to place buttons - Adding rocker on/off switch - Switching LED terminal blocks to .1" headers 2021-06-24: Revision 9 - Moving to nrf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"
- note removed: "Revision history: 2022-04-12: Revision 11 - Switching boost converter and inductor 2022-03-11: Revision 10 - Adding second tactile switch - Adjusting board dimensions to place buttons - Adding rocker on/off switch - Switching LED terminal blocks to .1" headers 2021-06-24: Revision 9 - Moving to nrf52840-DK BSP pins for buttons and leds - Driving LEDs with active LOW - Adding debugging pins for sw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"

Commit message: Bigger resistor array
Parts:
- RN2: DIGIKEY YC124J-1.0KCT-ND -> YC324J-1.0KCT-ND
Changed lines of the file:
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@@
 </part>
 <part name="RN2" library="resistor-dil" library_urn="urn:adsk.eagle:library:342" deviceset="4R-N" device="EXBS8V" package3d_urn="urn:adsk.eagle:package:24925/1">
-<attribute name="DIGIKEY" value="YC124J-1.0KCT-ND"/>
+<attribute name="DIGIKEY" value="YC324J-1.0KCT-ND"/>
 </part>
 <part name="R1" library="SparkFun" deviceset="RESISTOR" device="0603-RES" value="100k">
